File: Arduino_Mega2560_Practice/Section_01_USB_ATmega16U2.kicad_sch (KiCad schematic)
At the start: 21 parts, among them J1 USB_C_Receptacle_USB2.0_16P, J2 Conn_02x03_Odd_Even, U1 ATMEGA16U2-MU, Y1 Crystal

Commit message: USB完成
Parts:
- added C7: 100nF, Capacitor_SMD:C_0603_1608Metric, symbol Arduino_Mega2560_Lib:C_SMD_0603
- added D1, D3: Yellow, LED_SMD:LED_0805_2012Metric, symbol Arduino_Mega2560_Lib:LED_0805
- added FID1, FID2, FID3, FID4: Fiducial, Fiducial:Fiducial_1mm_Mask3mm, symbol Mechanical:Fiducial
- added J3: Conn_02x02_Odd_Even, Arduino_Mega2560_FP:CONN_M20-9980245_HRW, symbol Arduino_Mega2560_Lib:Header_2x02
- added JP2: SolderJumper_2_Open, Jumper:SolderJumper-2_P1.3mm_Open_Pad1.0x1.5mm, symbol Arduino_Mega2560_Lib:SolderJumper_2
- added RN2: 22R, Resistor_SMD:R_Array_Convex_4x0612, symbol Device:R_Pack04_Split
- added RN3, RN4: 1K, Resistor_SMD:R_Array_Convex_4x0612, symbol Arduino_Mega2560_Lib:RArray_4x0612
Connections:
- net +5V: now also RN4.3 (R3.1), RN4.4 (R4.1)
- net GND: now also RN3.5 (R4.2)
- net RXL: now reaches U1.10 (PD4)
- net RXL: now also D3.1 (K)
- net TXL: now reaches U1.11 (PD5)
- net TXL: now also D1.1 (K)
- net at U1.13 (PD7): now also C7.1, RN3.4 (R4.1)
- net 8PB4: now reaches U1.18 (PB4)
- net 8PB4: now also J3.1 (Pin_1)
- net 8PB5: now reaches U1.19 (PB5)
- net 8PB5: now also J3.3 (Pin_3)
- net 8PB6: now reaches U1.20 (PB6)
- net 8PB6: now also J3.2 (Pin_2)
- net 8PB7: now reaches U1.21 (PB7)
- net 8PB7: now also J3.4 (Pin_4)
- net M8RXD: now reaches U1.8 (PD2)
- net M8RXD: now also U1.9 (PD3), RN4.7 (R2.2), RN4.8 (R1.2)
- new net: D3.2 (A), RN4.5 (R4.2)
- new net: D1.2 (A), RN4.6 (R3.2)
- new net PE0: RN4.2 (R2.1)
- new net PE1: RN4.1 (R1.1)
- new net RESET: C7.2, JP2.1 (A), JP2.2 (B)
- no-connect marks 2 -> 15

Commit message: USB完成2
Parts:
- added C11: 100n, Capacitor_SMD:C_0603_1608Metric, symbol Device:C
Connections:
- net +5V: now also C11.1
- net GND: now also C11.2
