File: Arduino_Mega2560_Practice/Section_03_Power_Supply.kicad_sch (KiCad schematic)
At the start: 0 parts

Commit message: P1
Parts:
- added C1, C2: 47uF, Arduino_Mega2560_FP:CAP_EEHZA1E470P, symbol Arduino_Mega2560_Lib:C_Pol
- added C12, C13, C17, C4, C6: 100nF, Capacitor_SMD:C_0603_1608Metric, symbol Arduino_Mega2560_Lib:C_SMD_0603
- added C16: 1uF, Capacitor_SMD:C_0603_1608Metric, symbol Arduino_Mega2560_Lib:C_SMD_0603
- added D4: D, Diode_SMD:D_SMB, symbol Arduino_Mega2560_Lib:D_SMB
- added D5: Yellow, LED_SMD:LED_0805_2012Metric, symbol Arduino_Mega2560_Lib:LED_0805
- added D6: Green, LED_SMD:LED_0805_2012Metric, symbol Arduino_Mega2560_Lib:LED_0805
- added J4: Barrel_Jack_Switch, Connector_BarrelJack:BarrelJack_Kycon_KLDX-0202-xC_Horizontal, symbol Arduino_Mega2560_Lib:Barrel_Jack_Switch
- added Q1: Q_PMOS_GSD, Package_TO_SOT_SMD:SC-59, symbol Arduino_Mega2560_Lib:Q_PMOS_GSD
- added RN6: 1k, Resistor_SMD:R_Array_Convex_4x0612, symbol Arduino_Mega2560_Lib:RArray_4x0612
- added RN7: 10k, Resistor_SMD:R_Array_Convex_4x0612, symbol Arduino_Mega2560_Lib:RArray_4x0612
- added U2: NCP1117-5.0_SOT223, Package_TO_SOT_SMD:SOT-223-3_TabPin2, symbol Arduino_Mega2560_Lib:NCP1117_5_0_SOT223
- added U6: LP2985-3.3, Package_TO_SOT_SMD:SOT-23-5, symbol Arduino_Mega2560_Lib:LP2985_3_3
- added U7: LMV358IDGKR, Package_SO:MSOP-8_3x3mm_P0.65mm, symbol Arduino_Mega2560_Lib:LMV358
Connections:
- new net: D4.2 (A), J4.1
- new net: D6.2 (A), RN6.1 (R1.1)
- new net: D5.2 (A), RN6.2 (R2.1)
- new net +3.3V: C16.1, U6.5 (VOUT), U7.6
- new net +5V: C13.1, C2.1, C6.1, Q1.2 (S), RN6.8 (R1.2), U2.2 (VO), U6.1 (VIN), U6.3 (ON/~{OFF}), U7.8 (VCC+)
- new net CMP: C17.1, RN7.5 (R4.2), RN7.6 (R3.2), U7.5
- new net GATE_CMD: Q1.1 (G), U7.7
- new net GND: C1.2, C12.2, C13.2, C16.2, C17.2, C2.2, C4.2, C6.2, D5.1 (K), D6.1 (K), J4.2, J4.3, RN7.4 (R4.1), U2.1 (GND), U6.2 (GND), U7.4 (GND)
- new net L13: RN6.7 (R2.2), U7.1, U7.2
- new net PB7: U7.3
- new net USBVCC: Q1.3 (D)
- new net VCC: C1.1, C12.1, C4.1, D4.1 (K), RN7.3 (R3.1), U2.3 (VI)
- no-connect marks 0 -> 1
